File: simple_pcb/SIO2Arduino.sch (EAGLE design)
At the start: 8 parts

Commit message: Updated PCB with version number. Fixed readme
Other:
- note added: "Simple PCB for SIO2Arduino. v1.2"
- note removed: "Simple PCB for SIO2Arduino."
Changed lines of the file:
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@@
 <plain>
 <text x="138.43" y="7.62" size="2.54" layer="94" align="top-left">Elias Zacarias</text>
-<text x="85.09" y="5.08" size="2.54" layer="94" align="top-left">Simple PCB for SIO2Arduino.</text>
+<text x="85.09" y="5.08" size="2.54" layer="94" align="top-left">Simple PCB for SIO2Arduino.
+v1.2</text>
 </plain>
 <instances>
@@
 </schematic>
 </drawing>
+<compatibility>
+<note version="6.3" minversion="6.2.2" severity="warning">
+Since Version 6.2.2 text objects can contain more than one line,
+which will not be processed correctly with this version.
+</note>
+</compatibility>
 </eagle>
